File: Schematic/MySensors_PIR/v1.1/MySensors_PIR.brd (EAGLE design)
At the start: 49.5 x 49.6 mm, 29 parts, among them IC1 5V, J0 JUMPER-PAD-2-NC_BY_TRACE, J1 JUMPER-PAD-2-NC_BY_TRACE, J2 JUMPER-PAD-3-2OF3_NC_BY_TRACE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, J3 JUMPER-PAD-3-2OF3_NC_BY_TRACE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, X1 Vin

Commit message: little changes
Parts:
- added T1, T2, T3, T4, T5, T6, T7, T8: LSP10, my:LSP10
Routing:
- net N$6: track 0.00 -> 9.75 mm
- net N$7: track 0.00 -> 7.11 mm
Changed lines of the file:
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@@
 <setting verticaltext="up"/>
 </settings>
-<grid distance="12.5" unitdist="mil" unit="mil" style="lines" multiple="1" display="yes" altdistance="0.025" altunitdist="inch" altunit="inch"/>
+<grid distance="3.125" unitdist="mil" unit="mil" style="lines" multiple="1" display="yes" altdistance="0.025" altunitdist="inch" altunit="inch"/>
 <layers>
 <layer number="1" name="Top" color="4" fill="1" visible="yes" active="yes"/>
@@
 <layer number="46" name="Milling" color="3" fill="1" visible="yes" active="yes"/>
 <layer number="47" name="Measures" color="7" fill="1" visible="yes" active="yes"/>
-<layer number="48" name="Document" color="7" fill="1" visible="no" active="yes"/>
+<layer number="48" name="Document" color="7" fill="1" visible="yes" active="yes"/>
 <layer number="49" name="Reference" color="7" fill="1" visible="yes" active="yes"/>
 <layer number="50" name="dxf" color="7" fill="1" visible="no" active="no"/>
@@
 <plain>
 <circle x="27.94" y="50.21" radius="30" width="0.0254" layer="47"/>
-<dimension x1="-12.7" y1="74.93" x2="-12.7" y2="25.4" x3="-8.382" y3="50.165" textsize="1.778" layer="48" dtype="diameter"/>
+<dimension x1="-12.7" y1="74.93" x2="-12.7" y2="25.4" x3="-8.382" y3="50.165" textsize="1.778" layer="48" dtype="diameter" visible="yes"/>
 <wire x1="13.97" y1="25.4" x2="16.256" y2="25.4" width="0" layer="20"/>
 <wire x1="16.256" y1="25.4" x2="16.256" y2="26.924" width="0" layer="20"/>
@@
 <wire x1="41.91" y1="74.93" x2="48.26" y2="68.58" width="0" layer="20"/>
 <wire x1="48.26" y1="68.58" x2="52.705" y2="62.23" width="0" layer="20"/>
-<dimension x1="3.175" y1="16.51" x2="52.705" y2="16.51" x3="27.94" y3="7.62" textsize="1.778" layer="48" dtype="diameter"/>
-<wire x1="27.94" y1="81.28" x2="27.94" y2="18.415" width="0" layer="48"/>
-<wire x1="62.23" y1="50.165" x2="-5.715" y2="50.165" width="0" layer="48"/>
-<dimension x1="62.23" y1="26.67" x2="62.25" y2="73.68" x3="66.0024375" y3="50.1734" textsize="1.778" layer="48" dtype="diameter"/>
-<dimension x1="-2.06" y1="50.21" x2="57.94" y2="50.21" x3="27.94" y3="86.36" textsize="1.778" layer="48" dtype="diameter"/>
-<dimension x1="-18.415" y1="46.99" x2="-18.415" y2="56.515" x3="-22.86" y3="51.7525" textsize="1.778" layer="48" dtype="diameter"/>
+<dimension x1="3.175" y1="16.51" x2="52.705" y2="16.51" x3="27.94" y3="10.874375" textsize="1.778" layer="48" dtype="diameter" visible="yes"/>
+<wire x1="27.94" y1="81.28" x2="27.94" y2="19.129375" width="0" layer="48"/>
+<wire x1="61.356875" y1="50.165" x2="-5.715" y2="50.165" width="0" layer="48"/>
+<dimension x1="62.23" y1="26.67" x2="62.25" y2="73.68" x3="66.0024375" y3="50.1734" textsize="1.778" layer="48" dtype="diameter" visible="yes"/>
+<dimension x1="-2.06" y1="50.21" x2="57.94" y2="50.21" x3="27.94" y3="83.185" textsize="1.778" layer="48" dtype="diameter" visible="yes"/>
+<dimension x1="-18.415" y1="48.10125" x2="-18.415" y2="51.626071875" x3="-15.5575" y3="49.863659375" textsize="1.778" layer="48" dtype="diameter" visible="yes"/>
 <hole x="7.62" y="50.165" drill="3.2"/>
 <hole x="48.26" y="50.165" drill="3.2"/>
-<dimension x1="8.89" y1="13.97" x2="46.99" y2="13.97" x3="27.94" y3="15.875" textsize="1.778" layer="48" dtype="diameter"/>
+<dimension x1="8.89" y1="13.97" x2="46.99" y2="13.97" x3="27.94" y3="16.271875" textsize="1.778" layer="48" dtype="diameter" visible="yes"/>
 <rectangle x1="46.3931" y1="57.8739" x2="46.4185" y2="57.8993" layer="22" rot="R180"/>
 <rectangle x1="46.2661" y1="57.8993" x2="46.4439" y2="57.9247" layer="22" rot="R180"/>
@@
 <text x="11.1125" y="39.0525" size="0.8128" layer="22" font="vector" rot="MR0">nc</text>
 <text x="11.1125" y="36.5125" size="0.8128" layer="22" font="vector" rot="MR0">dat</text>
-<text x="11.1125" y="33.9725" size="0.8128" layer="22" font="vector" rot="MR0">vcc</text>
+<text x="11.1125" y="33.893125" size="0.8128" layer="22" font="vector" rot="MR0">vcc</text>
 <text x="14.9225" y="29.5275" size="0.6096" layer="22" font="vector" rot="MR0">TX</text>
 <text x="17.4625" y="29.5275" size="0.6096" layer="22" font="vector" rot="MR0">RX</text>
@@
 </element>
 <element name="U$2" library="ohw-logo" package="OSHW_FILLX100_NOTEXT" value="" x="46.92" y="44.6975"/>
+<element name="T1" library="my" package="LSP10" value="LSP10" x="11.1125" y="50.165" smashed="yes" rot="R90">
+<attribute name="VALUE" x="10.8585" y="50.165" size="0.0254" layer="27" rot="R90"/>
+</element>
+<element name="T2" library="my" package="LSP10" value="LSP10" x="44.7675" y="50.165" smashed="yes" rot="R90">
+<attribute name="VALUE" x="44.5135" y="50.165" size="0.0254" layer="27" rot="R90"/>
+</element>
+<element name="T3" library="my" package="LSP10" value="LSP10" x="21.59" y="27.94" smashed="yes" rot="R90">
+<attribute name="VALUE" x="21.336" y="27.94" size="0.0254" layer="27" rot="R90"/>
+</element>
+<element name="T4" library="my" package="LSP10" value="LSP10" x="24.4475" y="27.94" smashed="yes" rot="R90">
+<attribute name="VALUE" x="24.1935" y="27.94" size="0.0254" layer="27" rot="R90"/>
+</element>
+<element name="T5" library="my" package="LSP10" value="LSP10" x="31.4325" y="27.94" smashed="yes" rot="R90">
+<attribute name="VALUE" x="31.1785" y="27.94" size="0.0254" layer="27" rot="R90"/>
+</element>
+<element name="T6" library="my" package="LSP10" value="LSP10" x="34.29" y="27.94" smashed="yes" rot="R90">
+<attribute name="VALUE" x="34.036" y="27.94" size="0.0254" layer="27" rot="R90"/>
+</element>
+<element name="T7" library="my" package="LSP10" value="LSP10" x="4.60375" y="50.165" smashed="yes" rot="R90">
+<attribute name="VALUE" x="4.34975" y="50.165" size="0.0254" layer="27" rot="R90"/>
+</element>
+<element name="T8" library="my" package="LSP10" value="LSP10" x="51.27625" y="50.165" smashed="yes" rot="R90">
+<attribute name="VALUE" x="51.02225" y="50.165" size="0.0254" layer="27" rot="R90"/>
+</element>
 </elements>
 <signals>
@@
 <via x="51.2445" y="38.4175" extent="1-16" drill="0.3048" shape="square"/>
 <via x="4.572" y="61.595" extent="1-16" drill="0.3048" shape="square"/>
+<via x="22.70125" y="53.34" extent="1-16" drill="0.3048" shape="square"/>
 </signal>
 <signal name="SDA">
@@
 <wire x1="8.89" y1="65.405" x2="9.30275" y2="65.88125" width="0.1524" layer="1"/>
 </signal>
+<signal name="N$6">
+<wire x1="33.3375" y1="46.910625" x2="33.734375" y2="46.910625" width="0.254" layer="1"/>
+<wire x1="33.734375" y1="46.910625" x2="35.08375" y2="48.339375" width="0.254" layer="1"/>
+<wire x1="35.08375" y1="48.339375" x2="40.9575" y2="48.339375" width="0.254" layer="1"/>
+<wire x1="40.9575" y1="48.339375" x2="41.989375" y2="47.228125" width="0.254" layer="1"/>
+</signal>
+<signal name="N$7">
+<wire x1="35.8775" y1="46.910625" x2="39.84625" y2="46.910625" width="0.254" layer="1"/>
+<wire x1="39.84625" y1="46.910625" x2="42.06875" y2="44.688125" width="0.254" layer="1"/>
+</signal>
 </signals>
+<errors>
+</errors>
 </board>
 </drawing>
