File: Schematic/MySensors_PIR/v1.1/MySensors_PIR.sch (EAGLE design)
At the start: 28 parts, among them IC1 5V, J0 JUMPER-PAD-2-NC_BY_TRACE, J1 JUMPER-PAD-2-NC_BY_TRACE, J2 JUMPER-PAD-3-2OF3_NC_BY_TRACE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, J3 JUMPER-PAD-3-2OF3_NC_BY_TRACE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, X1 Vin

Commit message: little changes
Parts:
- added T1, T2, T3, T4, T5, T6, T7, T8: LSP10, my:LSP10
Other:
- note added: "Dummy"
- moved on the sheet: A0, A1, A2, A3, ARDUINO, C1, C2, C4, D1, D5, D6, D7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
